Commit message: add lidar.xacro

File: description/properties.xacro (robot description, xacro)
@@ -3,14 +3,17 @@
     <!-- Color Definitions -->
     <material name="white">
-        <color rgba= "1 1 1 1"/>
+        <color rgba="1 1 1 1" />
     </material>
     <material name="orange">
-        <color rgba= "1 0.3 0.1 1"/>
+        <color rgba="1 0.3 0.1 1" />
     </material>
     <material name="blue">
-        <color rgba= "0.2 0.2 1 1"/>
+        <color rgba="0.2 0.2 1 1" />
     </material>
     <material name="black">
-        <color rgba= "0 0 0 1"/>
+        <color rgba="0 0 0 1" />
+    </material>
+    <material name="red">
+        <color rgba="1 0 0 1" />
     </material>
 </robot>

File: description/robot.urdf.xacro (robot description, xacro)
@@ -1,7 +1,8 @@
 <?xml version="1.0"?>
-<robot xmlns:xacro="http://www.ros.org/wiki/xacro"  name="robot">
+<robot xmlns:xacro="http://www.ros.org/wiki/xacro" name="robot">
     <!-- Example link -->
-    <xacro:include filename="properties.xacro"/>
-    <xacro:include filename="inertial_macros.xacro"/>
-    <xacro:include filename="robot_core.xacro"/>
+    <xacro:include filename="properties.xacro" />
+    <xacro:include filename="inertial_macros.xacro" />
+    <xacro:include filename="lidar.xacro" />
+    <xacro:include filename="robot_core.xacro" />
 </robot>
