Commit message: [UPDATE] Se agregaron los gazebo tags

File: description/robot_core.xacro (robot description, xacro)
@@ -29,4 +29,7 @@
         </xacro:inertial_box>
     </link>
+    <gazebo reference="chassis">
+        <material>Gazebo/White</material>
+    </gazebo>
  <!-- left wheel joint -->
     <joint name="left_wheel_joint" type="continuous">
@@ -53,4 +56,7 @@
         </xacro:inertial_cylinder>
     </link>
+    <gazebo reference="left_wheel">
+        <material>Gazebo/Blue</material>
+    </gazebo>
      <!-- right wheel joint -->
     <joint name="right_wheel_joint" type="continuous">
@@ -77,4 +83,7 @@
         </xacro:inertial_cylinder>
     </link>
+    <gazebo reference="right_wheel">
+        <material>Gazebo/Blue</material>
+    </gazebo>
      <!-- caster wheel joint -->
     <joint name="caster_wheel_joint" type="fixed">
@@ -83,5 +92,5 @@
         <origin xyz="0.24 0 0"/>
     </joint>
-<!-- left wheel link -->
+<!-- caster wheel link -->
     <link name="caster_wheel">
         <visual>
@@ -100,3 +109,8 @@
         </xacro:inertial_sphere>
     </link>
+    <gazebo reference="caster_wheel">
+        <material>Gazebo/Black</material>
+        <mu1 value = "0.001" />
+        <mu2 value = "0.001" />
+    </gazebo>
 </robot>
