Commit message: [ADD] Se agregaron los parámetros para el SLAM

File: description/robot.urdf.xacro (robot description, xacro)
@@ -4,5 +4,6 @@
     <xacro:include filename="properties.xacro" />
     <xacro:include filename="inertial_macros.xacro" />
+    <xacro:include filename="robot_core.xacro" />
+    <xacro:include filename="gazebo_control.xacro" />
     <xacro:include filename="lidar.xacro" />
-    <xacro:include filename="robot_core.xacro" />
 </robot>

File: description/robot_core.xacro (robot description, xacro)
@@ -10,4 +10,11 @@
         <origin xyz="-0.1 0 0"/>
     </joint>
+    <joint name="base_footprint_joint" type="fixed">
+        <parent link="base_link"/>
+        <child link="base_footprint"/>
+        <origin xyz="0 0 -0.025"/>
+    </joint>
+    <link name="base_footprint">
+    </link>
  <!-- chassis link -->
     <link name="chassis">

Commit message: Se agragan cambios

File: description/robot.urdf.xacro (robot description, xacro)
@@ -2,8 +2,9 @@
 <robot xmlns:xacro="http://www.ros.org/wiki/xacro" name="robot">
     <!-- Example link -->
-    <xacro:include filename="properties.xacro" />
-    <xacro:include filename="inertial_macros.xacro" />
-    <xacro:include filename="robot_core.xacro" />
-    <xacro:include filename="gazebo_control.xacro" />
-    <xacro:include filename="lidar.xacro" />
+    <xacro:include filename="properties.xacro"/>
+    <xacro:include filename="robot_core.xacro"/>
+    <xacro:include filename="inertial_macros.xacro"/>
+    <!-- <xacro:include filename="gazebo_control.xacro"/> -->
+    <xacro:include filename="ros2_control.xacro"/>
+    <xacro:include filename="lidar.xacro"/>
 </robot>

File: description/robot_core.xacro (robot description, xacro)
@@ -1,6 +1,7 @@
 <?xml version="1.0"?>
 <robot xmlns:xacro="http://www.ros.org/wiki/xacro">
+    <!-- Example link -->
     <xacro:include filename="inertial_macros.xacro"/>
- <!-- Example link -->
+    <!-- Example link -->
     <link name="base_link">
     </link>
@@ -10,12 +11,5 @@
         <origin xyz="-0.1 0 0"/>
     </joint>
-    <joint name="base_footprint_joint" type="fixed">
-        <parent link="base_link"/>
-        <child link="base_footprint"/>
-        <origin xyz="0 0 -0.025"/>
-    </joint>
-    <link name="base_footprint">
-    </link>
- <!-- chassis link -->
+    <!-- chassis link -->
     <link name="chassis">
         <visual>
@@ -39,5 +33,5 @@
         <material>Gazebo/White</material>
     </gazebo>
- <!-- left wheel joint -->
+    <!-- left wheel joint -->
     <joint name="left_wheel_joint" type="continuous">
         <parent link="base_link"/>
@@ -46,5 +40,5 @@
         <axis xyz="0 0 1"/>
     </joint>
- <!-- left wheel link -->
+    <!-- left wheel link -->
     <link name="left_wheel">
         <visual>
@@ -56,5 +50,5 @@
         <collision>
             <geometry>
-                <cylinder radius="0.05" length="0.04"/>
+                <sphere radius="0.05"/>
             </geometry>
         </collision>
@@ -66,5 +60,5 @@
         <material>Gazebo/Blue</material>
     </gazebo>
-     <!-- right wheel joint -->
+    <!-- right wheel joint -->
     <joint name="right_wheel_joint" type="continuous">
         <parent link="base_link"/>
@@ -81,7 +75,7 @@
             <material name="blue"/>
         </visual>
-        <collision>
+                <collision>
             <geometry>
-                <cylinder radius="0.05" length="0.04"/>
+                <sphere radius="0.05"/>
             </geometry>
         </collision>
@@ -93,5 +87,5 @@
         <material>Gazebo/Blue</material>
     </gazebo>
-     <!-- caster wheel joint -->
+    <!-- caster wheel joint -->
     <joint name="caster_wheel_joint" type="fixed">
         <parent link="chassis"/>
@@ -99,5 +93,5 @@
         <origin xyz="0.24 0 0"/>
     </joint>
-<!-- caster wheel link -->
+    <!-- caster wheel link -->
     <link name="caster_wheel">
         <visual>
@@ -121,3 +115,10 @@
         <mu2 value = "0.001" />
     </gazebo>
+    <joint name="base_footprint_joint" type="fixed">
+        <parent link="base_link"/>
+        <child link="base_footprint"/>
+        <origin xyz="0 0 -0.025"/>
+    </joint>
+    <link name="base_footprint">
+    </link>
 </robot>
