Commit message: [Update] Akckerman URDF

File: description/gazebo_control_akerman.xacro (robot description, xacro)
@@ -1,31 +1,46 @@
 <?xml version="1.0"?>
 <robot xmlns:xacro="http://www.ros.org/wiki/xacro">
-    <!-- Ackermann robot plugin -->
-    <gazebo>
-      <plugin name="ackermann_drive" filename="libgazebo_ros_ackermann_drive.so">
-          <!-- Steering joint -->
-          <steering_joint>steering_joint</steering_joint>
-          <front_left_wheel_joint>front_left_wheel_joint</front_left_wheel_joint>
-          <front_right_wheel_joint>front_right_wheel_joint</front_right_wheel_joint>
-          <rear_left_wheel_joint>rear_left_wheel_joint</rear_left_wheel_joint>
-          <rear_right_wheel_joint>rear_right_wheel_joint</rear_right_wheel_joint>
-          <!-- Wheel information -->
-          <wheel_base>0.35</wheel_base>
-          <track_width>0.3</track_width>
-          <wheel_radius>0.05</wheel_radius>
-          <!-- Max steering angle -->
-          <max_steering_angle>0.5</max_steering_angle>
-          <!-- Limits -->
-          <max_steering_torque>100</max_steering_torque>
-          <max_steering_rate>1.0</max_steering_rate>
-          <max_wheel_torque>200</max_wheel_torque>
-          <max_wheel_acceleration>10.0</max_wheel_acceleration>
-          <!-- Outputs -->
-          <odometry_frame>odom</odometry_frame>
-          <robot_base_frame>base_link</robot_base_frame>
-          <publish_odom>true</publish_odom>
-          <publish_odom_tf>true</publish_odom_tf>
-          <publish_wheel_tf>true</publish_wheel_tf>
-      </plugin>
+  <!-- Ackermann robot plugin -->
+  <gazebo>
+    <plugin name="gazebo_ros_ackermann_drive" filename="libgazebo_ros_ackermann_drive.so">
+      <!-- <ros>
+        <namespace>demo</namespace>
+        <remapping>cmd_vel:=cmd_demo</remapping>
+        <remapping>odom:=odom_demo</remapping>
+        <remapping>distance:=distance_demo</remapping>
+      </ros> -->
+      <update_rate>100.0</update_rate>
+      <!-- wheels -->
+      <front_left_wheel_joint>front_left_wheel_joint</front_left_wheel_joint>
+      <front_right_wheel_joint>front_right_wheel_joint</front_right_wheel_joint>
+      <front_left_joint>front_left_steer_joint</front_left_joint>
+      <front_right_joint>front_right_steer_joint</front_right_joint>
+      <rear_left_joint>rear_left_wheel_joint</rear_left_joint>
+      <rear_right_joint>rear_right_wheel_joint</rear_right_joint>
+      <left_steering_joint>front_left_steer_joint</left_steering_joint>
+      <right_steering_joint>front_right_steer_joint</right_steering_joint>
+      <steering_wheel_joint>steering_joint</steering_wheel_joint>
+      <!-- Max absolute steer angle for tyre in radians-->
+      <!-- Any cmd_vel angular z greater than this would be capped -->
+      <max_steer>0.6458</max_steer>
+      <!-- Max absolute steering angle of steering wheel -->
+      <max_steering_angle>7.85</max_steering_angle>
+      <!-- Max absolute linear speed in m/s -->
+      <max_speed>20</max_speed>
+      <!-- PID tuning -->
+      <left_steering_pid_gain>1500 0 1</left_steering_pid_gain>
+      <left_steering_i_range>0 0</left_steering_i_range>
+      <right_steering_pid_gain>1500 0 1</right_steering_pid_gain>
+      <right_steering_i_range>0 0</right_steering_i_range>
+      <linear_velocity_pid_gain>1000 0 1</linear_velocity_pid_gain>
+      <linear_velocity_i_range>0 0</linear_velocity_i_range>
+      <!-- output -->
+      <publish_odom>true</publish_odom>
+      <publish_odom_tf>true</publish_odom_tf>
+      <publish_wheel_tf>true</publish_wheel_tf>
+      <publish_distance>true</publish_distance>
+      <odometry_frame>odom</odometry_frame>
+      <robot_base_frame>base_footprint</robot_base_frame>
+    </plugin>
   </gazebo>
 </robot>

File: description/robot_akerman.urdf.xacro (robot description, xacro)
@@ -3,8 +3,7 @@
     <!-- Example link -->
     <xacro:include filename="properties.xacro" />
-    <xacro:include filename="robot_core.xacro" />
     <xacro:include filename="inertial_macros.xacro" />
-    <!-- <xacro:include filename="gazebo_control.xacro"/> -->
-    <xacro:include filename="ros2_control.xacro" />
-    <xacro:include filename="lidar.xacro" />
+    <xacro:include filename="robot_core_akerman.xacro" />
+    <xacro:include filename="gazebo_control_akerman.xacro" />
+    <!-- <xacro:include filename="lidar.xacro" /> -->
 </robot>

File: description/robot_core.xacro (robot description, xacro)
@@ -2,30 +2,30 @@
 <robot xmlns:xacro="http://www.ros.org/wiki/xacro">
     <!-- Example link -->
-    <xacro:include filename="inertial_macros.xacro"/>
+    <xacro:include filename="inertial_macros.xacro" />
     <!-- Example link -->
     <link name="base_link">
     </link>
     <joint name="base_link" type="fixed">
-        <parent link="base_link"/>
-        <child link="chassis"/>
-        <origin xyz="-0.1 0 0"/>
+        <parent link="base_link" />
+        <child link="chassis" />
+        <origin xyz="-0.1 0 0" />
     </joint>
     <!-- chassis link -->
     <link name="chassis">
         <visual>
-            <origin xyz="0.15 0 0.075"/>
+            <origin xyz="0.15 0 0.075" />
             <geometry>
-                <box size="0.3 0.3 0.15"/>
+                <box size="0.3 0.3 0.15" />
             </geometry>
-            <material name="white"/>
+            <material name="white" />
         </visual>
         <collision>
-            <origin xyz="0.15 0 0.075"/>
+            <origin xyz="0.15 0 0.075" />
             <geometry>
-                <box size="0.3 0.3 0.15"/>
+                <box size="0.3 0.3 0.15" />
             </geometry>
         </collision>
         <xacro:inertial_box mass="0.5" x="0.3" y="0.3" z="0.15">
-            <origin xyz="0.15 0 0.075" rpy="0 0 0"/>
+            <origin xyz="0.15 0 0.075" rpy="0 0 0" />
         </xacro:inertial_box>
     </link>
@@ -35,8 +35,8 @@
     <!-- left wheel joint -->
     <joint name="left_wheel_joint" type="continuous">
-        <parent link="base_link"/>
-        <child link="left_wheel"/>
-        <origin xyz="0 0.175 0" rpy="-${pi/2} 0 0"/>
-        <axis xyz="0 0 1"/>
+        <parent link="base_link" />
+        <child link="left_wheel" />
+        <origin xyz="0 0.175 0" rpy="-${pi/2} 0 0" />
+        <axis xyz="0 0 1" />
     </joint>
     <!-- left wheel link -->
@@ -44,15 +44,15 @@
         <visual>
             <geometry>
-                <cylinder radius="0.05" length="0.04"/>
+                <cylinder radius="0.05" length="0.04" />
             </geometry>
-            <material name="blue"/>
+            <material name="blue" />
         </visual>
         <collision>
             <geometry>
-                <sphere radius="0.05"/>
+                <sphere radius="0.05" />
             </geometry>
         </collision>
         <xacro:inertial_cylinder mass="0.1" length="0.04" radius="0.05">
-            <origin xyz="0 0 0" rpy="0 0 0"/>
+            <origin xyz="0 0 0" rpy="0 0 0" />
         </xacro:inertial_cylinder>
     </link>
@@ -62,8 +62,8 @@
     <!-- right wheel joint -->
     <joint name="right_wheel_joint" type="continuous">
-        <parent link="base_link"/>
-        <child link="right_wheel"/>
-        <origin xyz="0 -0.175 0" rpy="${pi/2} 0 0"/>
-        <axis xyz="0 0 -1"/>
+        <parent link="base_link" />
+        <child link="right_wheel" />
+        <origin xyz="0 -0.175 0" rpy="${pi/2} 0 0" />
+        <axis xyz="0 0 -1" />
     </joint>
     <!-- right wheel link -->
@@ -71,15 +71,15 @@
         <visual>
             <geometry>
-                <cylinder radius="0.05" length="0.04"/>
+                <cylinder radius="0.05" length="0.04" />
             </geometry>
-            <material name="blue"/>
+            <material name="blue" />
         </visual>
-                <collision>
+        <collision>
             <geometry>
-                <sphere radius="0.05"/>
+                <sphere radius="0.05" />
             </geometry>
         </collision>
         <xacro:inertial_cylinder mass="0.1" length="0.04" radius="0.05">
-            <origin xyz="0 0 0" rpy="0 0 0"/>
+            <origin xyz="0 0 0" rpy="0 0 0" />
         </xacro:inertial_cylinder>
     </link>
@@ -89,7 +89,7 @@
     <!-- caster wheel joint -->
     <joint name="caster_wheel_joint" type="fixed">
-        <parent link="chassis"/>
-        <child link="caster_wheel"/>
-        <origin xyz="0.24 0 0"/>
+        <parent link="chassis" />
+        <child link="caster_wheel" />
+        <origin xyz="0.24 0 0" />
     </joint>
     <!-- caster wheel link -->
@@ -97,26 +97,26 @@
         <visual>
             <geometry>
-                <sphere radius="0.05"/>
+                <sphere radius="0.05" />
             </geometry>
-            <material name="black"/>
+            <material name="black" />
         </visual>
         <collision>
             <geometry>
-                <sphere radius="0.05"/>
+                <sphere radius="0.05" />
             </geometry>
         </collision>
         <xacro:inertial_sphere mass="0.1" radius="0.05">
-            <origin xyz="0 0 0" rpy="0 0 0"/>
+            <origin xyz="0 0 0" rpy="0 0 0" />
         </xacro:inertial_sphere>
     </link>
     <gazebo reference="caster_wheel">
         <material>Gazebo/Black</material>
-        <mu1 value = "0.001" />
-        <mu2 value = "0.001" />
+        <mu1 value="0.001" />
+        <mu2 value="0.001" />
     </gazebo>
     <joint name="base_footprint_joint" type="fixed">
-        <parent link="base_link"/>
-        <child link="base_footprint"/>
-        <origin xyz="0 0 -0.025"/>
+        <parent link="base_link" />
+        <child link="base_footprint" />
+        <origin xyz="0 0 -0.025" />
     </joint>
     <link name="base_footprint">

File: description/robot_core_akerman.xacro (robot description, xacro)
@@ -1,184 +1,202 @@
+<?xml version="1.0"?>
 <robot xmlns:xacro="http://www.ros.org/wiki/xacro">
-    <!-- Include Inertial Macros -->
-    <xacro:include filename="inertial_macros.xacro"/>
-    <!-- Base link -->
+    <!-- Example link -->
+    <xacro:include filename="inertial_macros.xacro" />
+    <!-- Example link -->
     <link name="base_link">
     </link>
     <joint name="base_link" type="fixed">
-        <parent link="base_link"/>
-        <child link="chassis"/>
-        <origin xyz="-0.1 0 0"/>
-    </joint>
-    <joint name="base_footprint_joint" type="fixed">
-        <parent link="base_link"/>
-        <child link="base_footprint"/>
-        <origin xyz="0 0 -0.025"/>
-    </joint>
-    <link name="base_footprint">
-    </link>
+        <parent link="base_link" />
+        <child link="chassis" />
+        <origin xyz="-0.1 0 0" />
+    </joint>
     <!-- chassis link -->
     <link name="chassis">
         <visual>
-            <origin xyz="0 0 0"/>
-            <geometry>
-                <box size="0.3 0.3 0.15"/>
-            </geometry>
-            <material name="white"/>
-        </visual>
-        <collision>
-            <origin xyz="0 0 0"/>
-            <geometry>
-                <box size="0.3 0.3 0.15"/>
+            <origin xyz="0.15 0 0.075" />
+            <geometry>
+                <box size="0.3 0.3 0.15" />
+            </geometry>
+            <material name="white" />
+        </visual>
+        <collision>
+            <origin xyz="0.15 0 0.075" />
+            <geometry>
+                <box size="0.3 0.3 0.15" />
             </geometry>
         </collision>
         <xacro:inertial_box mass="0.5" x="0.3" y="0.3" z="0.15">
-            <origin xyz="0 0 0" rpy="0 0 0"/>
+            <origin xyz="0.15 0 0.075" rpy="0 0 0" />
         </xacro:inertial_box>
     </link>
-    <gazebo reference="chassis">
+    <gazebo
+        reference="chassis">
         <material>Gazebo/White</material>
     </gazebo>
-    <!-- front left wheel joint -->
+    <!-- left wheel link -->
+    <link name="rear_left_wheel">
+        <visual>
+            <geometry>
+                <cylinder radius="0.05" length="0.04" />
+            </geometry>
+            <material name="blue" />
+        </visual>
+        <collision>
+            <geometry>
+                <sphere radius="0.05" />
+            </geometry>
+        </collision>
+        <xacro:inertial_cylinder mass="0.1" length="0.04" radius="0.05">
+            <origin xyz="0 0 0" rpy="0 0 0" />
+        </xacro:inertial_cylinder>
+    </link>
+    <gazebo
+        reference="rear_left_wheel">
+        <material>Gazebo/blue</material>
+    </gazebo>
+    <!-- right wheel link -->
+    <link name="rear_right_wheel">
+        <visual>
+            <geometry>
+                <cylinder radius="0.05" length="0.04" />
+            </geometry>
+            <material name="blue" />
+        </visual>
+        <collision>
+            <geometry>
+                <sphere radius="0.05" />
+            </geometry>
+        </collision>
+        <xacro:inertial_cylinder mass="0.1" length="0.04" radius="0.05">
+            <origin xyz="0 0 0" rpy="0 0 0" />
+        </xacro:inertial_cylinder>
+    </link>
+    <gazebo
+        reference="rear_right_wheel">
+        <material>Gazebo/blue</material>
+    </gazebo>
+    <link name="front_right_wheel">
+        <visual>
+            <geometry>
+                <cylinder radius="0.05" length="0.04" />
+            </geometry>
+            <material name="blue" />
+        </visual>
+        <collision>
+            <geometry>
+                <sphere radius="0.05" />
+            </geometry>
+        </collision>
+        <xacro:inertial_cylinder mass="0.1" length="0.04" radius="0.05">
+            <origin xyz="0 0 0" rpy="0 0 0" />
+        </xacro:inertial_cylinder>
+    </link>
+    <gazebo
+        reference="front_right_wheel">
+        <material>Gazebo/blue</material>
+    </gazebo>
+    <link name="front_left_wheel">
+        <visual>
+            <geometry>
+                <cylinder radius="0.05" length="0.04" />
+            </geometry>
+            <material name="blue" />
+        </visual>
+        <collision>
+            <geometry>
+                <sphere radius="0.05" />
+            </geometry>
+        </collision>
+        <xacro:inertial_cylinder mass="0.1" length="0.04" radius="0.05">
+            <origin xyz="0 0 0" rpy="0 0 0" />
+        </xacro:inertial_cylinder>
+    </link>
+    <gazebo
+        reference="front_left_wheel">
+        <material>Gazebo/blue</material>
+    </gazebo>
+    <!-- Steering wheel link -->
+    <link name="steering_wheel">
+        <visual>
+            <origin xyz="0 0 0.02" />
+            <geometry>
+                <cylinder radius="0.03" length="0.04" />
+            </geometry>
+            <material name="red" />
+        </visual>
+        <collision>
+            <origin xyz="0 0 0.02" />
+            <geometry>
+                <cylinder radius="0.03" length="0.04" />
+            </geometry>
+        </collision>
+        <xacro:inertial_cylinder mass="0.05" length="0.04" radius="0.03">
+            <origin xyz="0 0 0.02" rpy="0 0 0" />
+        </xacro:inertial_cylinder>
+    </link>
+    <!-- right wheel joint -->
+    <joint name="rear_right_wheel_joint"
+        type="continuous">
+        <parent link="base_link" />
+        <child link="rear_right_wheel" />
+        <origin xyz="0 -0.175 0" rpy="${pi/2} 0 0" />
+        <axis xyz="0 0 -1" />
+    </joint>
+    <!-- left wheel joint -->
+    <joint name="rear_left_wheel_joint"
+        type="continuous">
+        <parent link="base_link" />
+        <child link="rear_left_wheel" />
+        <origin xyz="0 0.175 0" rpy="-${pi/2} 0 0" />
+        <axis xyz="0 0 1" />
+    </joint>
+    <!-- Conectar el steering_wheel al chasis -->
+    <joint name="steering_joint" type="revolute">
+        <parent link="base_link" />
+        <child link="steering_wheel" />
+        <origin xyz="0.20 0 0.02" />
+        <axis xyz="0 0 1" />
+        <limit effort="100" lower="-0.5" upper="0.5" velocity="1" />
+    </joint>
+    <link name="right_steering_link"></link>
+    <link name="left_steering_link"></link>
+    <!-- Conectar right_steering_link al steering_wheel -->
+    <joint
+        name="front_right_steer_joint" type="revolute">
+        <parent link="steering_wheel" />
+        <child link="right_steering_link" />
+        <origin xyz="0 -0.175 0" />
+        <axis xyz="0 0 1" />
+        <limit effort="100" lower="-0.5" upper="0.5" velocity="1" />
+    </joint>
+    <!-- Conectar left_steering_link al steering_wheel -->
+    <joint name="front_left_steer_joint" type="revolute">
+        <parent link="steering_wheel" />
+        <child link="left_steering_link" />
+        <origin xyz="0  0.175 0" />
+        <axis xyz="0 0 1" />
+        <limit effort="100" lower="-0.5" upper="0.5" velocity="1" />
+    </joint>
+    <!-- Conectar el right_steering_link a la llanta delantera derecha -->
+    <joint
+        name="front_right_wheel_joint" type="continuous">
+        <parent link="right_steering_link" />
+        <child link="front_right_wheel" />
+        <origin xyz="0 0 -0.01" rpy="-${pi/2} 0 0" />
+        <axis xyz="0 0 -1" />
+    </joint>  <!-- Conectar el left_steering_link a la llanta delantera
+    izquierda -->
     <joint name="front_left_wheel_joint" type="continuous">
-        <parent link="base_link"/>
-        <child link="front_left_wheel"/>
-        <origin xyz="0 0.175 0" rpy="-${pi/2} 0 0"/>
-        <axis xyz="0 0 1"/>
-    </joint>
-    <!-- front left wheel link -->
-    <link name="front_left_wheel">
-        <visual>
-            <origin xyz="0 0 0"/>
-            <geometry>
-                <cylinder radius="0.05" length="0.04"/>
-            </geometry>
-            <material name="blue"/>
-        </visual>
-        <collision>
-            <origin xyz="0 0 0"/>
-            <geometry>
-                <cylinder radius="0.05" length="0.04"/>
-            </geometry>
-        </collision>
-        <xacro:inertial_cylinder mass="0.1" length="0.04" radius="0.05">
-            <origin xyz="0 0 0" rpy="0 0 0"/>
-        </xacro:inertial_cylinder>
-    </link>
-    <gazebo reference="front_left_wheel">
-        <material>Gazebo/Blue</material>
-    </gazebo>
-    <!-- front right wheel joint -->
-    <joint name="front_right_wheel_joint" type="continuous">
-        <parent link="base_link"/>
-        <child link="front_right_wheel"/>
-        <origin xyz="0 -0.175 0" rpy="${pi/2} 0 0"/>
-        <axis xyz="0 0 -1"/>
-    </joint>
-    <!-- front right wheel link -->
-    <link name="front_right_wheel">
-        <visual>
-            <origin xyz="0 0 0"/>
-            <geometry>
-                <cylinder radius="0.05" length="0.04"/>
-            </geometry>
-            <material name="blue"/>
-        </visual>
-        <collision>
-            <origin xyz="0 0 0"/>
-            <geometry>
-                <cylinder radius="0.05" length="0.04"/>
-            </geometry>
-        </collision>
-        <xacro:inertial_cylinder mass="0.1" length="0.04" radius="0.05">
-            <origin xyz="0 0 0" rpy="0 0 0"/>
-        </xacro:inertial_cylinder>
-    </link>
-    <gazebo reference="front_right_wheel">
-        <material>Gazebo/Blue</material>
-    </gazebo>
-    <!-- rear left wheel joint -->
-    <joint name="rear_left_wheel_joint" type="continuous">
-        <parent link="base_link"/>
-        <child link="rear_left_wheel"/>
-        <origin xyz="0.1 0.175 0" rpy="-${pi/2} 0 0"/>
-        <axis xyz="0 0 1"/>
-    </joint>
-    <!-- rear left wheel link -->
-    <link name="rear_left_wheel">
-        <visual>
-            <origin xyz="0 0 0"/>
-            <geometry>
-                <cylinder radius="0.05" length="0.04"/>
-            </geometry>
-            <material name="blue"/>
-        </visual>
-        <collision>
-            <origin xyz="0 0 0"/>
-            <geometry>
-                <cylinder radius="0.05" length="0.04"/>
-            </geometry>
-        </collision>
-        <xacro:inertial_cylinder mass="0.1" length="0.04" radius="0.05">
-            <origin xyz="0 0 0" rpy="0 0 0"/>
-        </xacro:inertial_cylinder>
-    </link>
-    <gazebo reference="rear_left_wheel">
-        <material>Gazebo/Blue</material>
-    </gazebo>
-    <!-- rear right wheel joint -->
-    <joint name="rear_right_wheel_joint" type="continuous">
-        <parent link="base_link"/>
-        <child link="rear_right_wheel"/>
-        <origin xyz="0.1 -0.175 0" rpy="${pi/2} 0 0"/>
-        <axis xyz="0 0 -1"/>
-    </joint>
-    <!-- rear right wheel link -->
-    <link name="rear_right_wheel">
-        <visual>
-            <origin xyz="0 0 0"/>
-            <geometry>
-                <cylinder radius="0.05" length="0.04"/>
-            </geometry>
-            <material name="blue"/>
-        </visual>
-        <collision>
-            <origin xyz="0 0 0"/>
-            <geometry>
-                <cylinder radius="0.05" length="0.04"/>
-            </geometry>
-        </collision>
-        <xacro:inertial_cylinder mass="0.1" length="0.04" radius="0.05">
-            <origin xyz="0 0 0" rpy="0 0 0"/>
-        </xacro:inertial_cylinder>
-    </link>
-    <gazebo reference="rear_right_wheel">
-        <material>Gazebo/Blue</material>
-    </gazebo>
-    <!-- Ackermann steering joint -->
-    <joint name="steering_joint" type="revolute">
-        <parent link="chassis"/>
-        <child link="steering_link"/>
-        <origin xyz="0 0 0.075"/>
-        <axis xyz="0 0 1"/>
-        <limit effort="100" lower="-0.5" upper="0.5" velocity="1"/>
-    </joint>
-    <!-- Steering link -->
-    <link name="steering_link">
-        <visual>
-            <origin xyz="0 0 0"/>
-            <geometry>
-                <box size="0.1 0.05 0.02"/>
-            </geometry>
-            <material name="gray"/>
-        </visual>
-        <collision>
-            <origin xyz="0 0 0"/>
-            <geometry>
-                <box size="0.1 0.05 0.02"/>
-            </geometry>
-        </collision>
-    </link>
-    <gazebo reference="steering_link">
-        <material>Gazebo/Gray</material>
-    </gazebo>
+        <parent link="left_steering_link" />
+        <child link="front_left_wheel" />
+        <origin xyz="0 0 -0.01" rpy="-${pi/2} 0 0" />
+        <axis xyz="0 0 1" />
+    </joint>
+    <joint name="base_footprint_joint" type="fixed">
+        <parent link="base_link" />
+        <child link="base_footprint" />
+        <origin xyz="0 0 -0.025" />
+    </joint>
+    <link name="base_footprint">
+    </link>
 </robot>
